File: Cubic2023_DCMotorDriver/Cubic2023_DCMotorDriver.kicad_sch (KiCad schematic)
At the start: 135 parts, among them IC1 A3921KLPTR-T, IC2 A3921KLPTR-T, IC3 BD63150AFM-E2, J1 Motor, J10 Conn_01x02_Male, J2 Motor, J3 Conn_01x04, J4 Motor, J6 Conn_02x07_Odd_Even, J7 Conn_02x07_Odd_Even, J8 Conn_02x07_Odd_Even, J9 Conn_01x02_Male, Q1 RJ1L12BGN, Q2 RJ1L12BGN, Q3 RJ1L12BGN, Q4 RJ1L12BGN, Q5 RJ1L12BGN, Q6 RJ1L12BGN, Q7 RJ1L12BGN, Q8 RJ1L12BGN, U1 ACS712ELCTR-30A-T, U2 ACS712ELCTR-30A-T

Commit message: WIP
Parts:
- D18, D2, D8: value SMBJ45CA -> SMBJ28CA
Other:
- note added: "connecter"
- note added: "pull down"
- moved on the sheet: C1, C10, C11, C12, C13, C14, C15, C16, C17, C18, C19, C2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

Commit message: WIP
Other:
- note added: "BD63150"
- note added: "Dead Time 2300ns"
- note added: "V5 Circuit"
- note added: "for motor connection"
- note added: "pull up"
- moved on the sheet: C5, D11, D16, D3, D4, D5, D6, D8, F1, IC3, J1, J10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

Commit message: WIP
Other:
- note added: "PS"
- note added: "VREF"
- note added: "VREF = 0.4V, 3A"
- note added: "error lamp"
- note added: "for solenoid valve"
- note removed: "VREF = 0.4, 3A"
- moved on the sheet: C12, C14, D1, D17, D19, D20, D7, F1, J10, J9, R14, R4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
