File: Cubic2023_Shield/Cubic2023_Shield.kicad_sch (KiCad schematic)
At the start: 138 parts, among them J1 Conn_01x06_Male, J10 Conn_02x06_Odd_Even, J11 Conn_01x07_Male, J12 Conn_01x07_Male, J13 Conn_01x06_Male, J14 Conn_01x06_Male, J15 Conn_02x06_Odd_Even, J16 Conn_02x06_Odd_Even, J17 Conn_01x02, J18 Conn_02x06_Odd_Even, J19 Conn_01x07_Male, J2 Conn_02x06_Odd_Even, J20 Conn_01x07_Male, J21 Conn_01x06_Male, J22 Conn_02x06_Odd_Even, J23 Conn_01x06_Male, J24 Conn_01x07_Male, J25 Conn_01x07_Male, J27 Conn_02x06_Odd_Even, J28 Conn_02x06_Odd_Even, J3 Conn_01x06_Male, J4 Conn_01x06, J5 Conn_01x06, J6 Conn_01x07_Male, J7 Conn_01x07_Male, J8 Conn_01x06_Male, J9 Conn_01x06_Male, U1 74VHC14, U2 74VHC14, U3 74VHC14, U4 74VHC14, U5 74LVC125

Commit message: WIP
Other:
- note added: "absolute encoder cognition"
- note added: "decoupling capacitor"
- note added: "encoder pull up"
- note added: "increment RP2040"
- note added: "increment connecter"
- note added: "increment encoder cognition"
- note added: "inverter"
- moved on the sheet: A1, C1, C2, C3, C4, C5, C69, C70, C71, C72, C73, C74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

Commit message: WIP
Connections:
- net ON renamed enable
Other:
- note added: "3-state buffer"
- note added: "Arduino nano 33 BLE"
- note added: "absolute RP2040"
- note added: "absolute connecter"
- note added: "emergency shutdown"
- note added: "to MotherBoard"
- moved on the sheet: A1, D10, D11, D12, D13, D14, D15, D16, D17, D9, J11, J12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
